Commit message: fixed launch & xacro

File: src/planning/urdf/main_car/car.xacro (robot description, xacro)
@@ -1,8 +1,9 @@
-<!--整车-->
+<!-- 整车 -->
 <robot xmlns:xacro="http://www.ros.org/wiki/xacro" name="main_car">
-    <xacro:property name="PI" value="3.141592653" />
-    <!-- 子文件包含 -->
-    <xacro:include filename="car_base.xacro" />
-    <xacro:include filename="car_camera.xacro" />
-    <xacro:include filename="car_radar.xacro" />
+    <!-- PI -->
+    <xacro:property name="PI" value="3.141592653"/>
+    <!-- 包含子文件, 要在参数定义之后, 子文件才能使用父文件的参数 -->
+    <xacro:include filename="car_base.xacro"/>
+    <xacro:include filename="car_camera.xacro"/>
+    <xacro:include filename="car_radar.xacro"/>
 </robot>

File: src/planning/urdf/main_car/car_base.xacro (robot description, xacro)
@@ -1,41 +1,39 @@
-<!--底盘-->
+<!-- 底盘 -->
 <robot xmlns:xacro="http://www.ros.org/wiki/xacro">
-    <!--车体-->
-    <xacro:property name="car_blength" value="3.0" />
-    <xacro:property name="car_width" value="1.5" />
-    <xacro:property name="car_height" value="0.6" />
-    <!--离地间隙-->
-    <xacro:property name="ground_height" value="0.2" />
-    <!--车轮-->
-    <xacro:include filename="car_wheels.xacro" />
-    <!--颜色-->
+    <!-- 车体尺寸 -->
+    <xacro:property name="car_length" value="3.0"/>
+    <xacro:property name="car_width" value="1.5"/>
+    <xacro:property name="car_height" value="0.6"/>
+    <!-- 离地间隙 -->
+    <xacro:property name="ground_height" value="0.2"/>
+    <!-- 包含子文件, 要在参数定义之后, 子文件才能使用父文件的参数 -->
+    <xacro:include filename="car_wheels.xacro"/>
+    <!-- 颜色 -->
     <material name="yellow">
-        <color rgba="0.9 0.6 0.0 0.7" />
+        <color rgba="0.9 0.6 0.0 0.7"/>
     </material>
-    <!--根坐标-->
-    <link name="map">
-    </link>
-    <!--底盘投影-->
-    <link name="base_footprint">
-    </link>
-    <!--底盘-->
+    <!-- 根坐标 -->
+    <link name="map"/>
+    <!-- 底盘在map的投影点 -->
+    <link name="base_footprint"/>
+    <!-- 底盘 -->
     <link name="base_link">
         <visual>
             <geometry>
-                <box size="${car_length} ${car_width} ${car_height}" />
+                <box size="${car_length} ${car_width} ${car_height}"/>
             </geometry>
-            <material name="yellow" />
+            <material name="yellow"/>
         </visual>
     </link>
-    <!--投影点关联到地图-->
+    <!-- 投影点关联到地图 -->
     <joint name="footprint_to_map" type="fixed">
-        <parent link="map" />
-        <child link="base_footprint" />
+        <parent link="map"/>
+        <child link="base_footprint"/>
     </joint>
-    <!--底盘关联到投影点-->
+    <!-- 底盘关联到投影点 -->
     <joint name="base_to_footprint" type="fixed">
-        <parent link="base_footprint" />
-        <child link="base_link" />
-        <origin xyz="0 0 ${car_height / 2.0 + ground_height}" />
+        <parent link="base_footprint"/>
+        <child link="base_link"/>
+        <origin xyz="0.0 0.0 ${car_height / 2.0 + ground_height}"/>
     </joint>
 </robot>

File: src/planning/urdf/main_car/car_camera.xacro (robot description, xacro)
@@ -1,30 +1,30 @@
-<!-- 文件名：camera_model.xacro -->
+<!-- 摄像头 -->
 <robot xmlns:xacro="http://www.ros.org/wiki/xacro">
-  <!-- 摄像头尺寸 -->
-  <xacro:property name="camera_length" value="0.1"/>
-  <xacro:property name="camera_width" value="0.8"/>
-  <xacro:property name="camera_height" value="0.2"/>
-  <!-- 摄像头偏移量 -->
-  <xacro:property name="camera_joint_x" value="${car_length / 2.0 - 0.02}"/>
-  <xacro:property name="camera_joint_y" value="0.0"/>
-  <xacro:property name="camera_joint_z" value="${camera_height / 2.0 + camera_height / 2.0}"/>
-  <!-- 颜色 -->
-  <material name="red">
-    <color rgba="1.0 0.0 0.0 0.8"/>
-  </material>
-  <!-- 摄像头几何 -->
-  <link name="camera">
-    <visual>
-      <geometry>
-        <box size="${camera_length} ${camera_width} ${camera_height}"/>
-      </geometry>
-      <material name="red"/>
-    </visual>
-  </link>
-  <!-- 摄像头关联到 base_link -->
-  <joint name="camera2base_joint" type="fixed">
-    <parent link="base_link"/>
-    <child link="camera"/>
-    <origin xyz="${camera_joint_x} ${camera_joint_y} ${camera_joint_z}"/>
-  </joint>
+    <!-- 摄像头尺寸 -->
+    <xacro:property name="camera_length" value="0.1"/>
+    <xacro:property name="camera_width" value="0.8"/>
+    <xacro:property name="camera_height" value="0.2"/>
+    <!-- 摄像头偏移量 -->
+    <xacro:property name="camera_joint_x" value="${car_length / 2.0 - 0.02}"/>
+    <xacro:property name="camera_joint_y" value="0.0"/>
+    <xacro:property name="camera_joint_z" value="${car_height / 2.0 + camera_height / 2.0}"/>
+    <!-- 颜色 -->
+    <material name="red">
+        <color rgba="1.0 0.0 0.0 0.8"/>
+    </material>
+    <!-- 摄像头几何 -->
+    <link name="camera">
+        <visual>
+            <geometry>
+                <box size="${camera_length} ${camera_width} ${camera_height}"/>
+            </geometry>
+            <material name="red"/>
+        </visual>
+    </link>
+    <!-- 摄像头关联到base_link -->
+    <joint name="camera2base_link" type="fixed">
+        <parent link="base_link"/>
+        <child link="camera"/>
+        <origin xyz="${camera_joint_x} ${camera_joint_y} ${camera_joint_z}"/>
+    </joint>
 </robot>

File: src/planning/urdf/main_car/car_radar.xacro (robot description, xacro)
@@ -1,29 +1,29 @@
-<!-- 文件名：radar_model.xacro -->
+<!-- 雷达 -->
 <robot xmlns:xacro="http://www.ros.org/wiki/xacro">
-  <!-- 雷达尺寸 -->
-  <xacro:property name="radar_radius" value="0.2"/>
-  <xacro:property name="radar_height" value="0.2"/>
-  <!-- 雷达偏移量 -->
-  <xacro:property name="radar_joint_x" value="0.0"/>
-  <xacro:property name="radar_joint_y" value="0.0"/>
-  <xacro:property name="radar_joint_z" value="${car_height / 2.0 + radar_height / 2.0}"/>
-  <!-- 颜色定义 -->
-  <material name="blue">
-    <color rgba="0.2 0.0 0.7 0.8"/>
-  </material>
-  <!-- 雷达几何 -->
-  <link name="radar">
-    <visual>
-      <geometry>
-        <cylinder radius="${radar_radius}" length="${radar_height}"/>
-      </geometry>
-      <material name="blue"/>
-    </visual>
-  </link>
-  <!-- 雷达关联到 base_link -->
-  <joint name="radar_joint" type="fixed">
-    <parent link="base_link"/>
-    <child link="radar"/>
-    <origin xyz="${radar_joint_x} ${radar_joint_y} ${radar_joint_z}"/>
-  </joint>
+    <!-- 雷达尺寸 -->
+    <xacro:property name="radar_radius" value="0.2"/>
+    <xacro:property name="radar_height" value="0.2"/>
+    <!-- 雷达偏移量 -->
+    <xacro:property name="radar_joint_x" value="0.0"/>
+    <xacro:property name="radar_joint_y" value="0.0"/>
+    <xacro:property name="radar_joint_z" value="${car_height / 2.0 + radar_height / 2.0}"/>
+    <!-- 颜色 -->
+    <material name="blue">
+        <color rgba="0.2 0.0 0.7 0.8"/>
+    </material>
+    <!-- 雷达几何 -->
+    <link name="radar">
+        <visual>
+            <geometry>
+                <cylinder radius="${radar_radius}" length="${radar_height}"/>
+            </geometry>
+            <material name="blue"/>
+        </visual>
+    </link>
+    <!-- 雷达关联到base_link -->
+    <joint name="radar2base_link" type="fixed">
+        <parent link="base_link"/>
+        <child link="radar"/>
+        <origin xyz="${radar_joint_x} ${radar_joint_y} ${radar_joint_z}"/>
+    </joint>
 </robot>

File: src/planning/urdf/main_car/car_wheels.xacro (robot description, xacro)
@@ -1,10 +1,10 @@
-<!-- 文件名：car_wheels.xacro -->
+<!-- 车轮 -->
 <robot xmlns:xacro="http://www.ros.org/wiki/xacro">
     <!-- 车轮尺寸 -->
-    <xacro:property name="wheel_radius" value="￥{car_height/2.0 + wheel_joint_z +ground_height}"/>
+    <xacro:property name="wheel_radius" value="${car_height / 2.0 + wheel_joint_z + ground_height}"/>
     <xacro:property name="wheel_width" value="0.3"/>
     <!-- 车轮偏移量 -->
     <xacro:property name="wheel_joint_x" value="${car_length / 2.0 - 0.4}"/>
-    <xacro:property name="wheel_joint_y" value="${car_width/2.0 + wheel_width / 2.0 + 0.1}"/>
+    <xacro:property name="wheel_joint_y" value="${car_width / 2.0 + wheel_width/ 2.0 + 0.1}"/>
     <xacro:property name="wheel_joint_z" value="-0.2"/>
     <!-- 颜色 -->
@@ -12,21 +12,21 @@
         <color rgba="0.0 0.0 0.0 0.7"/>
     </material>
-    <!-- 车轮几何 this is a function -->
+    <!-- 车轮几何 -->
     <xacro:macro name="wheel_geometry" params="wheel_name">
         <link name="${wheel_name}">
-        <visual>
-            <geometry>
-            <cylinder radius="${wheel_radius}" length="${wheel_width}"/>
-            </geometry>
-            <origin rpy="${PI/2.0} 0.0 0.0"/>
-            <material name="black"/>
-        </visual>
+            <visual>
+                <geometry>
+                    <cylinder radius="${wheel_radius}" length="${wheel_width}"/>
+                </geometry>
+                <origin rpy="${PI / 2.0} 0.0 0.0"/>
+                <material name="black"/>
+            </visual>
         </link>
     </xacro:macro>
     <!-- 后轮函数 -->
-    <xacro:macro name="wheel_rgar_func" params="wheel_name left_flag">
+    <xacro:macro name="wheel_rear_func" params="wheel_name left_flag">
         <!-- 车轮几何 -->
         <xacro:wheel_geometry wheel_name="${wheel_name}"/>
-        <!-- 车轮关联到 base_link -->
+        <!-- 车轮关联到base_link -->
         <joint name="${wheel_name}_rolling" type="continuous">
             <parent link="base_link"/>
@@ -38,9 +38,9 @@
     <!-- 前轮函数 -->
     <xacro:macro name="wheel_front_func" params="wheel_name left_flag">
-        <!-- 1. 车轮几何 -->
+        <!-- 车轮几何 -->
         <xacro:wheel_geometry wheel_name="${wheel_name}"/>
-        <!-- 2. 转向节几何 -->
+        <!-- 转向节几何 -->
         <link name="${wheel_name}_steering_knuckle"/>
-        <!-- 3. 转向节关联到 base_link（转向关节） -->
+        <!-- 转向节关联到base_link -->
         <joint name="${wheel_name}_turning" type="revolute">
             <parent link="base_link"/>
@@ -48,7 +48,7 @@
             <origin xyz="${wheel_joint_x} ${wheel_joint_y * left_flag} ${wheel_joint_z}"/>
             <axis xyz="0 0 1"/>
-            <limit effort="0.0" velocity="0.0" lower="${-PI/6.0}" upper="${PI/6.0}"/>
+            <limit effort="0.0" velocity="0.0" lower="-${PI / 6.0}" upper="${PI / 6.0}" />
         </joint>
-        <!-- 4. 车轮关联到转向节（滚动关节） -->
+        <!-- 车轮关联到转向节 -->
         <joint name="${wheel_name}_rolling" type="continuous">
             <parent link="${wheel_name}_steering_knuckle"/>
@@ -58,5 +58,5 @@
         </joint>
     </xacro:macro>
-    <!-- create 车轮 -->
+    <!-- 生成4个车轮 -->
     <xacro:wheel_front_func wheel_name="left_front" left_flag="1"/>
     <xacro:wheel_front_func wheel_name="right_front" left_flag="-1"/>
